File: PCB/boost_regulator_MIC2288.sch (EAGLE design)
At the start: 13 parts, among them U1 MIC2288YD5-TR

Commit message: Changed resistor values, edited description
Parts:
- R1: value 40K -> 47K
- R2: value 4K7 -> 5K1
Changed lines of the file:
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@@
 <part name="P+3" library="supply1" library_urn="urn:adsk.eagle:library:371" deviceset="VCC/2" device=""/>
 <part name="GND3" library="supply1" library_urn="urn:adsk.eagle:library:371" deviceset="GND" device=""/>
-<part name="R1" library="52101-101-REV-A" library_urn="urn:adsk.eagle:library:15662110" deviceset="RC-MASTER-SMD_R_" device="0603MP" package3d_urn="urn:adsk.eagle:package:15662272/2" value="40K"/>
-<part name="R2" library="52101-101-REV-A" library_urn="urn:adsk.eagle:library:15662110" deviceset="RC-MASTER-SMD_R_" device="0603MP" package3d_urn="urn:adsk.eagle:package:15662272/2" value="4K7"/>
+<part name="R1" library="52101-101-REV-A" library_urn="urn:adsk.eagle:library:15662110" deviceset="RC-MASTER-SMD_R_" device="0603MP" package3d_urn="urn:adsk.eagle:package:15662272/2" value="47K"/>
+<part name="R2" library="52101-101-REV-A" library_urn="urn:adsk.eagle:library:15662110" deviceset="RC-MASTER-SMD_R_" device="0603MP" package3d_urn="urn:adsk.eagle:package:15662272/2" value="5K1"/>
 <part name="C_CO2" library="SparkFun-Capacitors" library_urn="urn:adsk.eagle:library:21100215" deviceset="22UF-POLAR" device="-PANASONIC_C-35V-20%" package3d_urn="urn:adsk.eagle:package:21099999/2" value="47uF"/>
 <part name="C2" library="52101-101-REV-A" library_urn="urn:adsk.eagle:library:15662110" deviceset="RC-MASTER-SMD_C_" device="0603MP" package3d_urn="urn:adsk.eagle:package:15662234/2" value="10uF"/>
